File: glorious-lm1117.kicad_pcb (KiCad board)
At the start: 2 copper layers, 98.6 x 38.4 mm, 55 parts, among them J1 Conn_01x02, J2 USB_C_Receptacle_USB2.0, U1 LM1117-3.3, U10 LM1117-3.3, U11 LM1117-3.3, U12 LM1117-3.3, U13 LM1117-3.3, U14 LM1117-3.3, U15 LM1117-3.3, U16 LM1117-3.3, U17 LM1117-3.3, U18 LM1117-3.3, U19 LM1117-3.3, U2 LM1117-3.3, U20 LM1117-3.3, U21 LM1117-3.3, U22 LM1117-3.3, U23 LM1117-3.3, U24 LM1117-3.3, U25 LM1117-3.3, U26 LM1117-3.3, U27 LM1117-3.3, U28 LM1117-3.3, U29 LM1117-3.3, U3 LM1117-3.3, U30 LM1117-3.3, U31 LM1117-3.3, U32 LM1117-3.3, U33 LM1117-3.3, U34 LM1117-3.3, U35 LM1117-3.3, U36 LM1117-3.3, U37 LM1117-3.3, U38 LM1117-3.3, U39 LM1117-3.3, U4 LM1117-3.3, U40 LM1117-3.3, U5 LM1117-3.3, U6 LM1117-3.3, U7 LM1117-3.3, U8 LM1117-3.3, U9 LM1117-3.3

Commit message: finished?  needs more obnoxious silk perhaps?
Parts:
- added D1: LED_Small, LED_SMD:LED_0603_1608Metric, F.Cu at (207.4, 89.0)
- moved R2 87.2 mm to (121.2, 94.0), turned to 0 degrees
- moved R3 87.2 mm to (121.2, 92.3), turned to 0 degrees
- moved R1 4.67 mm to (207.4, 84.6), turned to -90 degrees
- moved J1 4.58 mm to (207.4, 80.1), turned to 180 degrees
- moved C4 2.95 mm to (204.8, 91.4)
- moved C2 2.95 mm to (204.8, 77.4)
- moved C6 2.95 mm to (204.8, 95.0)
- moved C8 2.95 mm to (204.8, 109.0)
- moved C10 0.57 mm to (121.4, 96.0), turned to 0 degrees
- moved C9 0.57 mm to (121.4, 90.4), turned to 0 degrees
Connections:
- R1 pad 2: GND -> Net-(R1-Pad2)
Routing:
- net GND: track 448.6 -> 534.4 mm, vias 38 -> 44
- net +5V: track 410.6 -> 476.9 mm, vias 38 -> 44
- net Net-(J1-Pad1): track 0.00 -> 3.70 mm
- net Net-(J2-PadB5): track 0.00 -> 2.86 mm
- net Net-(R1-Pad2): track 0.00 -> 2.79 mm
- net Net-(J2-PadA5): track 0.00 -> 2.65 mm
- net +3V3: track 446.5 -> 444.7 mm
- added copper zone on F.Cu, net +5V
- added copper zone on B.Cu, net GND
Other:
- board text added: "Glorious LM1117! Burning Iq for fun! Burning Iq for profit! false.ekta.is Jan 2022"
- board text added: "Look ma! Zero Load!"
- board text added: "{dblquote}Sponsors{dblquote} Steffanx ##GD32 formerly ##STM32 for chat professionals"
- board text removed: "Glorious LM1117 Iq for fun and profit"
- board text removed: "Sponsors: Steffanx"
