File: glorious-lm1117.kicad_sch (KiCad schematic)
At the start: 55 parts, among them J1 Conn_01x02, J2 USB_C_Receptacle_USB2.0, U1 LM1117-3.3, U10 LM1117-3.3, U11 LM1117-3.3, U12 LM1117-3.3, U13 LM1117-3.3, U14 LM1117-3.3, U15 LM1117-3.3, U16 LM1117-3.3, U17 LM1117-3.3, U18 LM1117-3.3, U19 LM1117-3.3, U2 LM1117-3.3, U20 LM1117-3.3, U21 LM1117-3.3, U22 LM1117-3.3, U23 LM1117-3.3, U24 LM1117-3.3, U25 LM1117-3.3, U26 LM1117-3.3, U27 LM1117-3.3, U28 LM1117-3.3, U29 LM1117-3.3, U3 LM1117-3.3, U30 LM1117-3.3, U31 LM1117-3.3, U32 LM1117-3.3, U33 LM1117-3.3, U34 LM1117-3.3, U35 LM1117-3.3, U36 LM1117-3.3, U37 LM1117-3.3, U38 LM1117-3.3, U39 LM1117-3.3, U4 LM1117-3.3, U40 LM1117-3.3, U5 LM1117-3.3, U6 LM1117-3.3, U7 LM1117-3.3, U8 LM1117-3.3, U9 LM1117-3.3

Commit message: finished?  needs more obnoxious silk perhaps?
Parts:
- added D1: LED_Small, LED_SMD:LED_0603_1608Metric, symbol Device:LED_Small
Connections:
- net GND: now also D1.1 (K); no longer R1.2
- new net: D1.2 (A), R1.2
Changed lines of the file:
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@@
-    (stroke (width 0) (type default) (color 0 0 0 0))
-  )
-  (wire (pts (xy 226.06 33.02) (xy 226.06 35.56))
     (stroke (width 0) (type default) (color 0 0 0 0))
   )
@@
     (stroke (width 0) (type default) (color 0 0 0 0))
   )
+  (wire (pts (xy 243.84 33.02) (xy 243.84 35.56))
+    (stroke (width 0) (type default) (color 0 0 0 0))
+  )
   (wire (pts (xy 185.42 132.08) (xy 187.96 132.08))
     (stroke (width 0) (type default) (color 0 0 0 0))
@@
     (stroke (width 0) (type default) (color 0 0 0 0))
   )
+  (wire (pts (xy 238.76 33.02) (xy 243.84 33.02))
+    (stroke (width 0) (type default) (color 0 0 0 0))
+  )
   (wire (pts (xy 25.4 55.88) (xy 22.86 55.88))
     (stroke (width 0) (type default) (color 0 0 0 0))
@@
   )
   (wire (pts (xy 73.66 116.84) (xy 71.12 116.84))
+    (stroke (width 0) (type default) (color 0 0 0 0))
+  )
+  (wire (pts (xy 226.06 33.02) (xy 233.68 33.02))
     (stroke (width 0) (type default) (color 0 0 0 0))
   )
@@
     (pin "1")
   )
-  (symbol (lib_id "power:GND") (at 226.06 35.56 0) (unit 1)
-    (in_bom yes) (on_board yes) (fields_autoplaced)
-    (property "Reference" "#PWR055" (id 0) (at 226.06 41.91 0)
-      (effects (font (size 1.27 1.27)) hide)
-    )
-    (property "Value" "GND" (id 1) (at 226.06 40.64 0))
-    (property "Footprint" "" (id 2) (at 226.06 35.56 0)
-      (effects (font (size 1.27 1.27)) hide)
-    )
-    (property "Datasheet" "" (id 3) (at 226.06 35.56 0)
+  (symbol (lib_id "power:GND") (at 243.84 35.56 0) (unit 1)
+    (in_bom yes) (on_board yes) (fields_autoplaced)
+    (property "Reference" "#PWR055" (id 0) (at 243.84 41.91 0)
+      (effects (font (size 1.27 1.27)) hide)
+    )
+    (property "Value" "GND" (id 1) (at 243.84 40.64 0))
+    (property "Footprint" "" (id 2) (at 243.84 35.56 0)
+      (effects (font (size 1.27 1.27)) hide)
+    )
+    (property "Datasheet" "" (id 3) (at 243.84 35.56 0)
       (effects (font (size 1.27 1.27)) hide)
     )
@@
     )
     (property "Datasheet" "~" (id 3) (at 165.1 30.48 0)
+      (effects (font (size 1.27 1.27)) hide)
+    )
+    (pin "1")
+    (pin "2")
+  )
+  (symbol (lib_id "Device:LED_Small") (at 236.22 33.02 180) (unit 1)
+    (in_bom yes) (on_board yes) (fields_autoplaced)
+    (property "Reference" "D1" (id 0) (at 236.1565 26.67 0))
+    (property "Value" "LED_Small" (id 1) (at 236.1565 29.21 0))
+    (property "Footprint" "LED_SMD:LED_0603_1608Metric" (id 2) (at 236.22 33.02 90)
+      (effects (font (size 1.27 1.27)) hide)
+    )
+    (property "Datasheet" "~" (id 3) (at 236.22 33.02 90)
       (effects (font (size 1.27 1.27)) hide)
     )
@@
       (reference "C10") (unit 1) (value "22uF") (footprint "Capacitor_SMD:C_0805_2012Metric")
     )
+    (path "/c32335a9-2bc8-4f58-b628-6f360a28a42c"
+      (reference "D1") (unit 1) (value "LED_Small") (footprint "LED_SMD:LED_0603_1608Metric")
+    )
     (path "/a2e7ee9f-2b22-4efc-bde3-6cb92221e200"
